File: Hardware/Digital_BuckBoost.kicad_sch (KiCad schematic)
At the start: 0 parts

Commit message: Modify the project name and page layout.
Other:
- title: (none) -> Digital_BuckBoost
Changed lines of the file:
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@@
 (kicad_sch (version 20211123) (generator eeschema)
   (paper "A4")
+  (title_block
+    (title "Digital_BuckBoost")
+    (date "2022-07-01")
+    (rev "1.0.1")
+  )
   (sheet (at 50.8 63.5) (size 25.4 38.1) (fields_autoplaced)
     (stroke (width 0.1524) (type solid) (color 0 0 0 0))
