File: Hardware/MCU.kicad_sch (KiCad schematic)
At the start: 5 parts

Commit message: Modify the project name and page layout.
Other:
- title: (none) -> Digital_BuckBoost
Changed lines of the file:
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@@
 (kicad_sch (version 20211123) (generator eeschema)
   (paper "A4")
+  (title_block
+    (title "Digital_BuckBoost")
+    (date "2022-07-01")
+    (rev "1.0.1")
+  )
   (symbol (lib_id "Integrated-circuit_micro-controller:HC32F460KEUA") (at 127 101.6 0) (unit 4)
     (in_bom yes) (on_board yes) (fields_autoplaced)
