File: Hardware/Main_Switcher.kicad_sch (KiCad schematic)
At the start: 5 parts

Commit message: Modify the project name and page layout.
Other:
- title: (none) -> Digital_BuckBoost
Changed lines of the file:
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@@
 (kicad_sch (version 20211123) (generator eeschema)
   (paper "A4")
+  (title_block
+    (title "Digital_BuckBoost")
+    (date "2022-07-01")
+    (rev "1.0.1")
+  )
   (symbol (lib_id "Power_transistor:HSBB4052") (at 152.4 101.6 0) (mirror y) (unit 1)
     (in_bom yes) (on_board yes) (fields_autoplaced)
