File: hardware/Main_Switcher.kicad_sch (KiCad schematic)
At the start: 5 parts

Commit message: Daily update
Parts:
- removed L?: Inductor, symbol Basic_passive_components:Inductor
- added L?: Power_Inductor, symbol Basic_passive_components:Power_Inductor
- Q? (x4): value HSBB4052 -> NTMFS5C670NL; footprint POWER_TRANSISTOR_SMD:SON-3333-FET -> POWER_TRANSISTOR_SMD:SON-8_5x6_M; symbol Power_transistor:HSBB4052 -> Power_transistor:NTMFS5C670NL
Connections:
- net at Q?.D (Drain): now also Q?.S (Source), L?.2
- net at Q?.S (Source): now also Q?.D (Drain), L?.1
Changed lines of the file:
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@@
     (rev "1.0.1")
   )
-  (symbol (lib_id "Power_transistor:HSBB4052") (at 152.4 101.6 0) (mirror y) (unit 1)
+  (junction (at 152.4 88.9) (diameter 0) (color 0 0 0 0)
+  )
+  (junction (at 101.6 88.9) (diameter 0) (color 0 0 0 0)
+  )
+  (wire (pts (xy 132.08 88.9) (xy 152.4 88.9))
+    (stroke (width 0) (type default) (color 0 0 0 0))
+  )
+  (wire (pts (xy 152.4 81.28) (xy 152.4 88.9))
+    (stroke (width 0) (type default) (color 0 0 0 0))
+  )
+  (wire (pts (xy 101.6 88.9) (xy 101.6 96.52))
+    (stroke (width 0) (type default) (color 0 0 0 0))
+  )
+  (wire (pts (xy 101.6 81.28) (xy 101.6 88.9))
+    (stroke (width 0) (type default) (color 0 0 0 0))
+  )
+  (wire (pts (xy 152.4 88.9) (xy 152.4 96.52))
+    (stroke (width 0) (type default) (color 0 0 0 0))
+  )
+  (wire (pts (xy 101.6 88.9) (xy 121.92 88.9))
+    (stroke (width 0) (type default) (color 0 0 0 0))
+  )
+  (symbol (lib_id "Power_transistor:NTMFS5C670NL") (at 152.4 101.6 0) (mirror y) (unit 1)
     (in_bom yes) (on_board yes) (fields_autoplaced)
     (property "Reference" "Q?" (id 0) (at 149.86 100.3299 0)
       (effects (font (size 1.27 1.27)) (justify left))
     )
-    (property "Value" "HSBB4052" (id 1) (at 149.86 102.8699 0)
+    (property "Value" "NTMFS5C670NL" (id 1) (at 149.86 102.8699 0)
       (effects (font (size 1.27 1.27)) (justify left))
     )
-    (property "Footprint" "POWER_TRANSISTOR_SMD:SON-3333-FET" (id 2) (at 130.81 97.79 0)
+    (property "Footprint" "POWER_TRANSISTOR_SMD:SON-8_5x6_M" (id 2) (at 130.81 97.79 0)
       (effects (font (size 1.27 1.27)) hide)
     )
@@
     (pin "S")
   )
-  (symbol (lib_id "Power_transistor:HSBB4052") (at 101.6 76.2 0) (unit 1)
+  (symbol (lib_id "Power_transistor:NTMFS5C670NL") (at 101.6 76.2 0) (unit 1)
     (in_bom yes) (on_board yes) (fields_autoplaced)
     (property "Reference" "Q?" (id 0) (at 104.14 74.9299 0)
       (effects (font (size 1.27 1.27)) (justify left))
     )
-    (property "Value" "HSBB4052" (id 1) (at 104.14 77.4699 0)
+    (property "Value" "NTMFS5C670NL" (id 1) (at 104.14 77.4699 0)
       (effects (font (size 1.27 1.27)) (justify left))
     )
-    (property "Footprint" "POWER_TRANSISTOR_SMD:SON-3333-FET" (id 2) (at 123.19 72.39 0)
+    (property "Footprint" "POWER_TRANSISTOR_SMD:SON-8_5x6_M" (id 2) (at 123.19 72.39 0)
       (effects (font (size 1.27 1.27)) hide)
     )
@@
     (pin "S")
   )
-  (symbol (lib_id "Power_transistor:HSBB4052") (at 152.4 76.2 0) (mirror y) (unit 1)
+  (symbol (lib_id "Power_transistor:NTMFS5C670NL") (at 152.4 76.2 0) (mirror y) (unit 1)
     (in_bom yes) (on_board yes) (fields_autoplaced)
     (property "Reference" "Q?" (id 0) (at 149.86 74.9299 0)
       (effects (font (size 1.27 1.27)) (justify left))
     )
-    (property "Value" "HSBB4052" (id 1) (at 149.86 77.4699 0)
+    (property "Value" "NTMFS5C670NL" (id 1) (at 149.86 77.4699 0)
       (effects (font (size 1.27 1.27)) (justify left))
     )
-    (property "Footprint" "POWER_TRANSISTOR_SMD:SON-3333-FET" (id 2) (at 130.81 72.39 0)
+    (property "Footprint" "POWER_TRANSISTOR_SMD:SON-8_5x6_M" (id 2) (at 130.81 72.39 0)
       (effects (font (size 1.27 1.27)) hide)
     )
@@
     (pin "S")
   )
-  (symbol (lib_id "Power_transistor:HSBB4052") (at 101.6 101.6 0) (unit 1)
+  (symbol (lib_id "Power_transistor:NTMFS5C670NL") (at 101.6 101.6 0) (unit 1)
     (in_bom yes) (on_board yes) (fields_autoplaced)
     (property "Reference" "Q?" (id 0) (at 104.14 100.3299 0)
       (effects (font (size 1.27 1.27)) (justify left))
     )
-    (property "Value" "HSBB4052" (id 1) (at 104.14 102.8699 0)
+    (property "Value" "NTMFS5C670NL" (id 1) (at 104.14 102.8699 0)
       (effects (font (size 1.27 1.27)) (justify left))
     )
-    (property "Footprint" "POWER_TRANSISTOR_SMD:SON-3333-FET" (id 2) (at 123.19 97.79 0)
+    (property "Footprint" "POWER_TRANSISTOR_SMD:SON-8_5x6_M" (id 2) (at 123.19 97.79 0)
       (effects (font (size 1.27 1.27)) hide)
     )
@@
     (pin "S")
   )
-  (symbol (lib_id "Basic_passive_components:Inductor") (at 127 88.9 0) (unit 1)
+  (symbol (lib_id "Basic_passive_components:Power_Inductor") (at 127 88.9 0) (unit 1)
     (in_bom yes) (on_board yes) (fields_autoplaced)
     (property "Reference" "L?" (id 0) (at 127 82.55 0))
-    (property "Value" "Inductor" (id 1) (at 127 85.09 0))
+    (property "Value" "Power_Inductor" (id 1) (at 127 85.09 0))
     (property "Footprint" "" (id 2) (at 127 88.9 0)
       (effects (font (size 1.27 1.27)) hide)
@@
     (pin "2")
   )
+  (symbol (lib_id "power:GND") (at 152.4 121.92 0) (unit 1)
+    (in_bom yes) (on_board yes) (fields_autoplaced)
+    (property "Reference" "#PWR?" (id 0) (at 152.4 128.27 0)
+      (effects (font (size 1.27 1.27)) hide)
+    )
+    (property "Value" "GND" (id 1) (at 152.4 127 0))
+    (property "Footprint" "" (id 2) (at 152.4 121.92 0)
+      (effects (font (size 1.27 1.27)) hide)
+    )
+    (property "Datasheet" "" (id 3) (at 152.4 121.92 0)
+      (effects (font (size 1.27 1.27)) hide)
+    )
+    (pin "1")
+  )
+  (symbol (lib_id "power:VDC") (at 101.6 50.8 0) (unit 1)
+    (in_bom yes) (on_board yes) (fields_autoplaced)
+    (property "Reference" "#PWR?" (id 0) (at 101.6 53.34 0)
+      (effects (font (size 1.27 1.27)) hide)
+    )
+    (property "Value" "VDC" (id 1) (at 101.6 45.72 0))
+    (property "Footprint" "" (id 2) (at 101.6 50.8 0)
+      (effects (font (size 1.27 1.27)) hide)
+    )
+    (property "Datasheet" "" (id 3) (at 101.6 50.8 0)
+      (effects (font (size 1.27 1.27)) hide)
+    )
+    (pin "1")
+  )
+  (symbol (lib_id "power:VBUS") (at 152.4 50.8 0) (unit 1)
+    (in_bom yes) (on_board yes) (fields_autoplaced)
+    (property "Reference" "#PWR?" (id 0) (at 152.4 54.61 0)
+      (effects (font (size 1.27 1.27)) hide)
+    )
+    (property "Value" "VBUS" (id 1) (at 152.4 45.72 0))
+    (property "Footprint" "" (id 2) (at 152.4 50.8 0)
+      (effects (font (size 1.27 1.27)) hide)
+    )
+    (property "Datasheet" "" (id 3) (at 152.4 50.8 0)
+      (effects (font (size 1.27 1.27)) hide)
+    )
+    (pin "1")
+  )
+  (symbol (lib_id "power:GND") (at 101.6 121.92 0) (unit 1)
+    (in_bom yes) (on_board yes) (fields_autoplaced)
+    (property "Reference" "#PWR?" (id 0) (at 101.6 128.27 0)
+      (effects (font (size 1.27 1.27)) hide)
+    )
+    (property "Value" "GND" (id 1) (at 101.6 127 0))
+    (property "Footprint" "" (id 2) (at 101.6 121.92 0)
+      (effects (font (size 1.27 1.27)) hide)
+    )
+    (property "Datasheet" "" (id 3) (at 101.6 121.92 0)
+      (effects (font (size 1.27 1.27)) hide)
+    )
+    (pin "1")
+  )
 )

Commit message: Update schematics.
Parts:
- added R?: Resistor, symbol Basic_passive_components:Resistor
Connections:
- net at Q?.D (Drain), Q?.S (Source): now also R?.2; no longer L?.2
- net BG2: now reaches Q?.G (Gate)
- net TG1: now reaches Q?.G (Gate)
- net TG2: now reaches Q?.G (Gate)
- net BG1: now reaches Q?.G (Gate)
- new net: L?.2, R?.1
Other:
- moved on the sheet: Q?
Changed lines of the file:
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@@
     (rev "1.0.1")
   )
-  (junction (at 152.4 88.9) (diameter 0) (color 0 0 0 0)
+  (junction (at 177.8 88.9) (diameter 0) (color 0 0 0 0)
   )
   (junction (at 101.6 88.9) (diameter 0) (color 0 0 0 0)
   )
-  (wire (pts (xy 132.08 88.9) (xy 152.4 88.9))
+  (wire (pts (xy 132.08 88.9) (xy 147.32 88.9))
     (stroke (width 0) (type default) (color 0 0 0 0))
   )
-  (wire (pts (xy 152.4 81.28) (xy 152.4 88.9))
+  (wire (pts (xy 177.8 81.28) (xy 177.8 88.9))
+    (stroke (width 0) (type default) (color 0 0 0 0))
+  )
+  (wire (pts (xy 182.88 76.2) (xy 193.04 76.2))
+    (stroke (width 0) (type default) (color 0 0 0 0))
+  )
+  (wire (pts (xy 157.48 88.9) (xy 177.8 88.9))
     (stroke (width 0) (type default) (color 0 0 0 0))
   )
@@
     (stroke (width 0) (type default) (color 0 0 0 0))
   )
+  (wire (pts (xy 86.36 101.6) (xy 96.52 101.6))
+    (stroke (width 0) (type default) (color 0 0 0 0))
+  )
+  (wire (pts (xy 86.36 76.2) (xy 96.52 76.2))
+    (stroke (width 0) (type default) (color 0 0 0 0))
+  )
   (wire (pts (xy 101.6 81.28) (xy 101.6 88.9))
     (stroke (width 0) (type default) (color 0 0 0 0))
   )
-  (wire (pts (xy 152.4 88.9) (xy 152.4 96.52))
+  (wire (pts (xy 177.8 88.9) (xy 177.8 96.52))
+    (stroke (width 0) (type default) (color 0 0 0 0))
+  )
+  (wire (pts (xy 182.88 101.6) (xy 193.04 101.6))
     (stroke (width 0) (type default) (color 0 0 0 0))
   )
@@
     (stroke (width 0) (type default) (color 0 0 0 0))
   )
-  (symbol (lib_id "Power_transistor:NTMFS5C670NL") (at 152.4 101.6 0) (mirror y) (unit 1)
+  (hierarchical_label "TG2" (shape input) (at 193.04 76.2 0)
+    (effects (font (size 1.27 1.27)) (justify left))
+  )
+  (hierarchical_label "TG1" (shape input) (at 86.36 76.2 180)
+    (effects (font (size 1.27 1.27)) (justify right))
+  )
+  (hierarchical_label "BG1" (shape input) (at 86.36 101.6 180)
+    (effects (font (size 1.27 1.27)) (justify right))
+  )
+  (hierarchical_label "BG2" (shape input) (at 193.04 101.6 0)
+    (effects (font (size 1.27 1.27)) (justify left))
+  )
+  (symbol (lib_id "Power_transistor:NTMFS5C670NL") (at 177.8 101.6 0) (mirror y) (unit 1)
     (in_bom yes) (on_board yes) (fields_autoplaced)
-    (property "Reference" "Q?" (id 0) (at 149.86 100.3299 0)
+    (property "Reference" "Q?" (id 0) (at 175.26 100.3299 0)
       (effects (font (size 1.27 1.27)) (justify left))
     )
-    (property "Value" "NTMFS5C670NL" (id 1) (at 149.86 102.8699 0)
+    (property "Value" "NTMFS5C670NL" (id 1) (at 175.26 102.8699 0)
       (effects (font (size 1.27 1.27)) (justify left))
     )
-    (property "Footprint" "POWER_TRANSISTOR_SMD:SON-8_5x6_M" (id 2) (at 130.81 97.79 0)
+    (property "Footprint" "POWER_TRANSISTOR_SMD:SON-8_5x6_M" (id 2) (at 156.21 97.79 0)
       (effects (font (size 1.27 1.27)) hide)
     )
-    (property "Datasheet" "" (id 3) (at 151.765 101.6 0)
+    (property "Datasheet" "" (id 3) (at 177.165 101.6 0)
       (effects (font (size 1.27 1.27)) hide)
     )
@@
     (pin "S")
   )
-  (symbol (lib_id "Power_transistor:NTMFS5C670NL") (at 152.4 76.2 0) (mirror y) (unit 1)
+  (symbol (lib_id "Power_transistor:NTMFS5C670NL") (at 177.8 76.2 0) (mirror y) (unit 1)
     (in_bom yes) (on_board yes) (fields_autoplaced)
-    (property "Reference" "Q?" (id 0) (at 149.86 74.9299 0)
+    (property "Reference" "Q?" (id 0) (at 175.26 74.9299 0)
       (effects (font (size 1.27 1.27)) (justify left))
     )
-    (property "Value" "NTMFS5C670NL" (id 1) (at 149.86 77.4699 0)
+    (property "Value" "NTMFS5C670NL" (id 1) (at 175.26 77.4699 0)
       (effects (font (size 1.27 1.27)) (justify left))
     )
-    (property "Footprint" "POWER_TRANSISTOR_SMD:SON-8_5x6_M" (id 2) (at 130.81 72.39 0)
+    (property "Footprint" "POWER_TRANSISTOR_SMD:SON-8_5x6_M" (id 2) (at 156.21 72.39 0)
       (effects (font (size 1.27 1.27)) hide)
     )
-    (property "Datasheet" "" (id 3) (at 151.765 76.2 0)
+    (property "Datasheet" "" (id 3) (at 177.165 76.2 0)
       (effects (font (size 1.27 1.27)) hide)
     )
@@
     (pin "2")
   )
-  (symbol (lib_id "power:GND") (at 152.4 121.92 0) (unit 1)
+  (symbol (lib_id "power:GND") (at 177.8 121.92 0) (unit 1)
     (in_bom yes) (on_board yes) (fields_autoplaced)
-    (property "Reference" "#PWR?" (id 0) (at 152.4 128.27 0)
+    (property "Reference" "#PWR?" (id 0) (at 177.8 128.27 0)
       (effects (font (size 1.27 1.27)) hide)
     )
-    (property "Value" "GND" (id 1) (at 152.4 127 0))
-    (property "Footprint" "" (id 2) (at 152.4 121.92 0)
+    (property "Value" "GND" (id 1) (at 177.8 127 0))
+    (property "Footprint" "" (id 2) (at 177.8 121.92 0)
       (effects (font (size 1.27 1.27)) hide)
     )
-    (property "Datasheet" "" (id 3) (at 152.4 121.92 0)
+    (property "Datasheet" "" (id 3) (at 177.8 121.92 0)
       (effects (font (size 1.27 1.27)) hide)
     )
@@
     (pin "1")
   )
-  (symbol (lib_id "power:VBUS") (at 152.4 50.8 0) (unit 1)
+  (symbol (lib_id "Basic_passive_components:Resistor") (at 152.4 88.9 0) (unit 1)
     (in_bom yes) (on_board yes) (fields_autoplaced)
-    (property "Reference" "#PWR?" (id 0) (at 152.4 54.61 0)
+    (property "Reference" "R?" (id 0) (at 152.4 82.55 0))
+    (property "Value" "Resistor" (id 1) (at 152.4 85.09 0))
+    (property "Footprint" "" (id 2) (at 148.59 85.09 0)
       (effects (font (size 1.27 1.27)) hide)
     )
-    (property "Value" "VBUS" (id 1) (at 152.4 45.72 0))
-    (property "Footprint" "" (id 2) (at 152.4 50.8 0)
+    (property "Datasheet" "" (id 3) (at 148.59 85.09 0)
       (effects (font (size 1.27 1.27)) hide)
     )
-    (property "Datasheet" "" (id 3) (at 152.4 50.8 0)
+    (pin "1")
+    (pin "2")
+  )
+  (symbol (lib_id "power:VBUS") (at 177.8 50.8 0) (unit 1)
+    (in_bom yes) (on_board yes) (fields_autoplaced)
+    (property "Reference" "#PWR?" (id 0) (at 177.8 54.61 0)
       (effects (font (size 1.27 1.27)) hide)
     )
+    (property "Value" "VBUS" (id 1) (at 177.8 45.72 0))
+    (property "Footprint" "" (id 2) (at 177.8 50.8 0)
+      (effects (font (size 1.27 1.27)) hide)
+    )
+    (property "Datasheet" "" (id 3) (at 177.8 50.8 0)
+      (effects (font (size 1.27 1.27)) hide)
+    )
