File: hardware/Digital_BuckBoost.kicad_sch (KiCad schematic)
At the start: 0 parts

Commit message: Nightly update
Update Driver and Main_Switch.
Other:
- sheet Main_Switcher renamed Main_Switch
- sheet Driver ports: added BG1, BG2, SW1, SW2, TG1, TG2; removed none
- sheet Main_Switch: file Main_Switcher.kicad_sch -> Main_Switch.kicad_sch
- sheet Main_Switch ports: added BG1, BG2, CS_N, CS_P, SW1, SW2, TG1, TG2; removed none

Commit message: Nightly update
Other:
- sheet Driver ports: added BS1, BS2, DRV1_EN, DRV2_EN, PWM1_H, PWM1_L, PWM2_H, PWM2_L; removed none
- sheet Main_Switch ports: added BS1, BS2, CS1_N, CS1_P, CS2_N, CS2_P; removed CS_N, CS_P

Commit message: Update Base_PWR
Other:
- sheet Base_PWR ports: added PW_DRV_EN; removed none
Changed lines of the file:
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@@
       (effects (font (size 1.27 1.27)) (justify left top))
+    )
+    (pin "PW_DRV_EN" input (at 76.2 152.4 0)
+      (effects (font (size 1.27 1.27)) (justify right))
     )
   )
