File: hardware/Digital_BuckBoost.kicad_sch (KiCad schematic)
At the start: 0 parts

Commit message: Nightly Update
Other:
- added sheet Amplifier (Amplifier.kicad_sch)

Commit message: Update schematics
Other:
- sheet MCU ports: added CAN_Rx, CAN_Tx, CS1_Buff, CS2_Buff, DRV1_EN, DRV2_EN, PWM1_H, PWM1_L, PWM2_H, PWM2_L, PW_DRV_EN, SWCLK, SWDIO, UART_Rx, UART_Tx; removed none

Commit message: Complete schematics
Other:
- sheet MCU ports: added none; removed CAN_Rx, CAN_Tx, SWCLK, SWDIO, UART_Rx, UART_Tx
