File: hardware/Amplifier.kicad_sch (KiCad schematic)
At the start: 12 parts

Commit message: Nightly update
Parts:
- removed C?: 100nF, 001_GN_RCL_SMD:C0402(1005M), symbol 001_Basic_PassiveComponents:101_Capacitor
- U? (x2): value MC4580G-K08 -> RS622XTDE8; footprint 003_GN_SMALL-SEMI_SMD:DFN-8_3020 -> 003_GN_SMALL-SEMI_SMD:DFN-8_2020; symbol 101_IntegratedCircuit_Amplifier:MC4580G-K08 -> 101_IntegratedCircuit_Amplifier:RS622XTDE8
Changed lines of the file:
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@@
     (effects (font (size 1.27 1.27)) (justify right))
   )
-  (symbol (lib_id "101_IntegratedCircuit_Amplifier:MC4580G-K08") (at 127 76.2 0) (unit 1)
-    (in_bom yes) (on_board yes) (fields_autoplaced)
-    (property "Reference" "U?" (id 0) (at 139.7 71.52 0))
-    (property "Value" "MC4580G-K08" (id 1) (at 139.7 74.06 0))
-    (property "Footprint" "003_GN_SMALL-SEMI_SMD:DFN-8_3020" (id 2) (at 149.225 67.31 0)
+  (symbol (lib_id "101_IntegratedCircuit_Amplifier:RS622XTDE8") (at 127 76.2 0) (unit 1)
+    (in_bom yes) (on_board yes) (fields_autoplaced)
+    (property "Reference" "U?" (id 0) (at 129.54 72.39 0))
+    (property "Value" "RS622XTDE8" (id 1) (at 134.62 69.85 0))
+    (property "Footprint" "003_GN_SMALL-SEMI_SMD:DFN-8_2020" (id 2) (at 147.32 67.31 0)
       (effects (font (size 1.27 1.27)) hide)
     )
@@
       (effects (font (size 1.27 1.27)) hide)
     )
-    (property "Symbol type" "Specified Device" (id 4) (at 138.43 64.77 0)
+    (property "Symbol type" "Specified Device" (id 4) (at 137.16 64.77 0)
       (effects (font (size 1.27 1.27)) hide)
     )
@@
     (pin "1")
   )
-  (symbol (lib_id "001_Basic_PassiveComponents:101_Capacitor") (at 177.8 127 90) (unit 1)
-    (in_bom yes) (on_board yes) (fields_autoplaced)
-    (property "Reference" "C?" (id 0) (at 180.34 125.7299 90)
-      (effects (font (size 1.27 1.27)) (justify right))
-    )
-    (property "Value" "100nF" (id 1) (at 180.34 128.2699 90)
-      (effects (font (size 1.27 1.27)) (justify right))
-    )
-    (property "Footprint" "001_GN_RCL_SMD:C0402(1005M)" (id 2) (at 177.8 127 0)
-      (effects (font (size 1.27 1.27)) hide)
-    )
-    (property "Datasheet" "" (id 3) (at 177.8 127 0)
-      (effects (font (size 1.27 1.27)) hide)
-    )
-    (property "Symbol type" "Alternate Source" (id 4) (at 172.72 127 0)
-      (effects (font (size 1.27 1.27)) hide)
-    )
-    (pin "1")
-    (pin "2")
-  )
   (symbol (lib_id "001_Basic_PassiveComponents:001_Resistor") (at 119.38 139.7 0) (unit 1)
     (in_bom yes) (on_board yes) (fields_autoplaced)
@@
     (pin "1")
   )
-  (symbol (lib_id "101_IntegratedCircuit_Amplifier:MC4580G-K08") (at 127 127 0) (unit 2)
-    (in_bom yes) (on_board yes) (fields_autoplaced)
-    (property "Reference" "U?" (id 0) (at 127 116.84 0))
-    (property "Value" "MC4580G-K08" (id 1) (at 127 119.38 0))
-    (property "Footprint" "003_GN_SMALL-SEMI_SMD:DFN-8_3020" (id 2) (at 149.225 118.11 0)
+  (symbol (lib_id "101_IntegratedCircuit_Amplifier:RS622XTDE8") (at 127 127 0) (unit 2)
+    (in_bom yes) (on_board yes) (fields_autoplaced)
+    (property "Reference" "U?" (id 0) (at 129.54 123.19 0))
+    (property "Value" "RS622XTDE8" (id 1) (at 134.62 120.65 0))
+    (property "Footprint" "003_GN_SMALL-SEMI_SMD:DFN-8_2020" (id 2) (at 147.32 118.11 0)
       (effects (font (size 1.27 1.27)) hide)
     )
@@
       (effects (font (size 1.27 1.27)) hide)
     )
-    (property "Symbol type" "Specified Device" (id 4) (at 138.43 115.57 0)
-      (effects (font (size 1.27 1.27)) hide)
-    )
+    (property "Symbol type" "Specified Device" (id 4) (at 137.16 115.57 0)
+      (effects (font (size 1.27 1.27)) hide)
+    )

Commit message: Update schematics
Parts:
- R? (x4): value 20kR -> 10kR
Changed lines of the file:
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@@
       (effects (font (size 1.27 1.27)) (justify right))
     )
-    (property "Value" "20kR" (id 1) (at 114.3 115.5699 90)
+    (property "Value" "10kR" (id 1) (at 114.3 115.5699 90)
       (effects (font (size 1.27 1.27)) (justify right))
     )
@@
     (in_bom yes) (on_board yes) (fields_autoplaced)
     (property "Reference" "R?" (id 0) (at 119.38 133.35 0))
-    (property "Value" "20kR" (id 1) (at 119.38 135.89 0))
+    (property "Value" "10kR" (id 1) (at 119.38 135.89 0))
     (property "Footprint" "001_GN_RCL_SMD:R0402(1005M)" (id 2) (at 115.57 135.89 0)
       (effects (font (size 1.27 1.27)) hide)
@@
     (in_bom yes) (on_board yes) (fields_autoplaced)
     (property "Reference" "R?" (id 0) (at 119.38 82.55 0))
-    (property "Value" "20kR" (id 1) (at 119.38 85.09 0))
+    (property "Value" "10kR" (id 1) (at 119.38 85.09 0))
     (property "Footprint" "001_GN_RCL_SMD:R0402(1005M)" (id 2) (at 115.57 85.09 0)
       (effects (font (size 1.27 1.27)) hide)
@@
       (effects (font (size 1.27 1.27)) (justify right))
     )
-    (property "Value" "20kR" (id 1) (at 114.3 64.7699 90)
-      (effects (font (size 1.27 1.27)) (justify right))
-    )
+    (property "Value" "10kR" (id 1) (at 114.3 64.7699 90)
+      (effects (font (size 1.27 1.27)) (justify right))
+    )

Commit message: Complete schematics
Parts:
- gave numbers to parts that had none: 10
Changed lines of the file:
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@@
   (symbol (lib_id "101_IntegratedCircuit_Amplifier:RS622XTDE8") (at 127 76.2 0) (unit 1)
     (in_bom yes) (on_board yes) (fields_autoplaced)
-    (property "Reference" "U?" (id 0) (at 129.54 72.39 0))
+    (property "Reference" "U7" (id 0) (at 129.54 72.39 0))
     (property "Value" "RS622XTDE8" (id 1) (at 134.62 69.85 0))
     (property "Footprint" "003_GN_SMALL-SEMI_SMD:DFN-8_2020" (id 2) (at 147.32 67.31 0)
@@
   (symbol (lib_id "PowerPort:GND") (at 127 93.98 0) (unit 1)
     (in_bom yes) (on_board yes) (fields_autoplaced)
-    (property "Reference" "#PWR?" (id 0) (at 127 100.33 0)
+    (property "Reference" "#PWR0192" (id 0) (at 127 100.33 0)
       (effects (font (size 1.27 1.27)) hide)
     )
@@
   (symbol (lib_id "001_Basic_PassiveComponents:001_Resistor") (at 111.76 114.3 90) (unit 1)
     (in_bom yes) (on_board yes) (fields_autoplaced)
-    (property "Reference" "R?" (id 0) (at 114.3 113.0299 90)
+    (property "Reference" "R40" (id 0) (at 114.3 113.0299 90)
       (effects (font (size 1.27 1.27)) (justify right))
     )
@@
   (symbol (lib_id "PowerPort:GND") (at 177.8 93.98 0) (unit 1)
     (in_bom yes) (on_board yes) (fields_autoplaced)
-    (property "Reference" "#PWR?" (id 0) (at 177.8 100.33 0)
+    (property "Reference" "#PWR0188" (id 0) (at 177.8 100.33 0)
       (effects (font (size 1.27 1.27)) hide)
     )
@@
   (symbol (lib_id "001_Basic_PassiveComponents:001_Resistor") (at 119.38 139.7 0) (unit 1)
     (in_bom yes) (on_board yes) (fields_autoplaced)
-    (property "Reference" "R?" (id 0) (at 119.38 133.35 0))
+    (property "Reference" "R42" (id 0) (at 119.38 133.35 0))
     (property "Value" "10kR" (id 1) (at 119.38 135.89 0))
     (property "Footprint" "001_GN_RCL_SMD:R0402(1005M)" (id 2) (at 115.57 135.89 0)
@@
   (symbol (lib_id "001_Basic_PassiveComponents:001_Resistor") (at 101.6 81.28 0) (unit 1)
     (in_bom yes) (on_board yes) (fields_autoplaced)
-    (property "Reference" "R?" (id 0) (at 101.6 74.93 0))
+    (property "Reference" "R36" (id 0) (at 101.6 74.93 0))
     (property "Value" "1kR" (id 1) (at 101.6 77.47 0))
     (property "Footprint" "001_GN_RCL_SMD:R0402(1005M)" (id 2) (at 97.79 77.47 0)
@@
   (symbol (lib_id "PowerPort:Vref") (at 111.76 55.88 0) (unit 1)
     (in_bom yes) (on_board yes) (fields_autoplaced)
-    (property "Reference" "#PWR?" (id 0) (at 106.68 59.69 0)
+    (property "Reference" "#PWR0186" (id 0) (at 106.68 59.69 0)
       (effects (font (size 1.27 1.27)) hide)
     )
@@
   (symbol (lib_id "001_Basic_PassiveComponents:001_Resistor") (at 119.38 88.9 0) (unit 1)
     (in_bom yes) (on_board yes) (fields_autoplaced)
-    (property "Reference" "R?" (id 0) (at 119.38 82.55 0))
+    (property "Reference" "R41" (id 0) (at 119.38 82.55 0))
     (property "Value" "10kR" (id 1) (at 119.38 85.09 0))
     (property "Footprint" "001_GN_RCL_SMD:R0402(1005M)" (id 2) (at 115.57 85.09 0)
@@
   (symbol (lib_id "001_Basic_PassiveComponents:001_Resistor") (at 101.6 132.08 0) (unit 1)
     (in_bom yes) (on_board yes) (fields_autoplaced)
-    (property "Reference" "R?" (id 0) (at 101.6 125.73 0))
+    (property "Reference" "R38" (id 0) (at 101.6 125.73 0))
     (property "Value" "1kR" (id 1) (at 101.6 128.27 0))
     (property "Footprint" "001_GN_RCL_SMD:R0402(1005M)" (id 2) (at 97.79 128.27 0)
@@
   (symbol (lib_id "001_Basic_PassiveComponents:001_Resistor") (at 101.6 121.92 0) (unit 1)
     (in_bom yes) (on_board yes) (fields_autoplaced)
-    (property "Reference" "R?" (id 0) (at 101.6 115.57 0))
+    (property "Reference" "R37" (id 0) (at 101.6 115.57 0))
     (property "Value" "1kR" (id 1) (at 101.6 118.11 0))
     (property "Footprint" "001_GN_RCL_SMD:R0402(1005M)" (id 2) (at 97.79 118.11 0)
@@
   (symbol (lib_id "001_Basic_PassiveComponents:101_Capacitor") (at 177.8 76.2 270) (unit 1)
     (in_bom yes) (on_board yes) (fields_autoplaced)
-    (property "Reference" "C?" (id 0) (at 180.34 74.9299 90)
+    (property "Reference" "C28" (id 0) (at 180.34 74.9299 90)
       (effects (font (size 1.27 1.27)) (justify left))
     )
@@
   (symbol (lib_id "power:+3V3") (at 127 55.88 0) (unit 1)
     (in_bom yes) (on_board yes) (fields_autoplaced)
-    (property "Reference" "#PWR?" (id 0) (at 127 59.69 0)
+    (property "Reference" "#PWR0187" (id 0) (at 127 59.69 0)
       (effects (font (size 1.27 1.27)) hide)
     )
@@
   (symbol (lib_id "101_IntegratedCircuit_Amplifier:RS622XTDE8") (at 127 127 0) (unit 2)
     (in_bom yes) (on_board yes) (fields_autoplaced)
-    (property "Reference" "U?" (id 0) (at 129.54 123.19 0))
+    (property "Reference" "U7" (id 0) (at 129.54 123.19 0))
     (property "Value" "RS622XTDE8" (id 1) (at 134.62 120.65 0))
     (property "Footprint" "003_GN_SMALL-SEMI_SMD:DFN-8_2020" (id 2) (at 147.32 118.11 0)
@@
   (symbol (lib_id "PowerPort:GND") (at 127 144.78 0) (unit 1)
     (in_bom yes) (on_board yes) (fields_autoplaced)
-    (property "Reference" "#PWR?" (id 0) (at 127 151.13 0)
+    (property "Reference" "#PWR0190" (id 0) (at 127 151.13 0)
       (effects (font (size 1.27 1.27)) hide)
     )
@@
   (symbol (lib_id "001_Basic_PassiveComponents:001_Resistor") (at 111.76 63.5 90) (unit 1)
     (in_bom yes) (on_board yes) (fields_autoplaced)
-    (property "Reference" "R?" (id 0) (at 114.3 62.2299 90)
+    (property "Reference" "R39" (id 0) (at 114.3 62.2299 90)
       (effects (font (size 1.27 1.27)) (justify right))
     )
@@
   (symbol (lib_id "001_Basic_PassiveComponents:001_Resistor") (at 101.6 71.12 0) (unit 1)
     (in_bom yes) (on_board yes) (fields_autoplaced)
-    (property "Reference" "R?" (id 0) (at 101.6 64.77 0))
+    (property "Reference" "R35" (id 0) (at 101.6 64.77 0))
     (property "Value" "1kR" (id 1) (at 101.6 67.31 0))
     (property "Footprint" "001_GN_RCL_SMD:R0402(1005M)" (id 2) (at 97.79 67.31 0)
@@
   (symbol (lib_id "PowerPort:Vref") (at 111.76 106.68 0) (unit 1)
     (in_bom yes) (on_board yes) (fields_autoplaced)
-    (property "Reference" "#PWR?" (id 0) (at 106.68 110.49 0)
+    (property "Reference" "#PWR0191" (id 0) (at 106.68 110.49 0)
       (effects (font (size 1.27 1.27)) hide)
     )
@@
   (symbol (lib_id "power:+3V3") (at 177.8 55.88 0) (unit 1)
     (in_bom yes) (on_board yes) (fields_autoplaced)
-    (property "Reference" "#PWR?" (id 0) (at 177.8 59.69 0)
-      (effects (font (size 1.27 1.27)) hide)
-    )
+    (property "Reference" "#PWR0189" (id 0) (at 177.8 59.69 0)
+      (effects (font (size 1.27 1.27)) hide)
+    )
