File: hardware/Driver.kicad_sch (KiCad schematic)
At the start: 0 parts

Commit message: Daily update
Parts:
- added U? (x2): DGD05473, GENERAL_SMALL-SEMI_SMD:DFN-3030_10, symbol Integrated-circuit_transistor_driver:DGD05473
Changed lines of the file:
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@@
     (rev "1.0.1")
   )
+  (symbol (lib_id "Integrated-circuit_transistor_driver:DGD05473") (at 101.6 127 0) (unit 1)
+    (in_bom yes) (on_board yes) (fields_autoplaced)
+    (property "Reference" "U?" (id 0) (at 101.6 113.03 0))
+    (property "Value" "DGD05473" (id 1) (at 101.6 115.57 0))
+    (property "Footprint" "GENERAL_SMALL-SEMI_SMD:DFN-3030_10" (id 2) (at 101.6 114.3 0)
+      (effects (font (size 1.27 1.27)) hide)
+    )
+    (property "Datasheet" "" (id 3) (at 101.6 121.92 0)
+      (effects (font (size 1.27 1.27)) hide)
+    )
+    (pin "1")
+    (pin "10")
+    (pin "2")
+    (pin "3")
+    (pin "4")
+    (pin "5")
+    (pin "6")
+    (pin "7")
+    (pin "8")
+    (pin "9")
+    (pin "EP")
+  )
+  (symbol (lib_id "Integrated-circuit_transistor_driver:DGD05473") (at 101.6 76.2 0) (unit 1)
+    (in_bom yes) (on_board yes) (fields_autoplaced)
+    (property "Reference" "U?" (id 0) (at 101.6 62.23 0))
+    (property "Value" "DGD05473" (id 1) (at 101.6 64.77 0))
+    (property "Footprint" "GENERAL_SMALL-SEMI_SMD:DFN-3030_10" (id 2) (at 101.6 63.5 0)
+      (effects (font (size 1.27 1.27)) hide)
+    )
+    (property "Datasheet" "" (id 3) (at 101.6 71.12 0)
+      (effects (font (size 1.27 1.27)) hide)
+    )
+    (pin "1")
+    (pin "10")
+    (pin "2")
+    (pin "3")
+    (pin "4")
+    (pin "5")
+    (pin "6")
+    (pin "7")
+    (pin "8")
+    (pin "9")
+    (pin "EP")
+  )
 )

Commit message: Nightly update
Update Driver and Main_Switch.
Parts:
- added C? (x2): 2.2uF, GENERAL_RCL_SMD:C0805(2012M), symbol Basic_passive_components:Capacitor
- added D? (x2): SS1060HEWS, POWER_DIODE_SMD:SOD-123HE, symbol Basic_semiconductor:Diode_Schottky
- added R? (x2): 3.3R, GENERAL_RCL_SMD:R0603(1608M), symbol Basic_passive_components:Resistor
Connections:
- net Vdrive: now reaches U?.1 (Vin)
- net Vdrive: now also U?.1 (Vin), D?.2 (Anode), D?.2 (Anode)
- net BG2: now reaches U?.10 (BG)
- net at U?.3 (BST): now also D?.1 (Cathode), R?.1 (x2)
- net TG2: now reaches U?.4 (TG)
- net SW2: now reaches U?.5 (SW)
- net SW2: now also C?.2
- net GND: now reaches U?.9 (GND)
- net GND: now also U?.9 (GND), U?.EP, U?.EP
- net BG1: now reaches U?.10 (BG)
- net TG1: now reaches U?.4 (TG)
- net SW1: now reaches U?.5 (SW)
- net SW1: now also C?.2
- new net: C?.1, R?.2 (x2)
Other:
- moved on the sheet: U?

Commit message: Nightly update
Parts:
- added R? (x2): 0R, 001_GN_RCL_SMD:R0603(1608M), symbol 001_Basic_PassiveComponents:001_Resistor
- C? (x2): symbol Basic_passive_components:Capacitor -> 001_Basic_PassiveComponents:101_Capacitor; Symbol type (none) -> Alternate Source
- D? (x2): symbol Basic_semiconductor:Diode_Schottky -> 002_Basic_SingleSemiconductor:002_Diode_Schottky; Symbol type (none) -> Alternate Source
- R? (x2): symbol Basic_passive_components:Resistor -> 001_Basic_PassiveComponents:001_Resistor; Symbol type (none) -> Alternate Source
- U? (x2): footprint GENERAL_SMALL-SEMI_SMD:DFN-3030_10 -> 003_GN_SMALL-SEMI_SMD:DFN-10_3030; symbol Integrated-circuit_transistor_driver:DGD05473 -> 105_IntegratedCircuit_TransistorDriver:DGD05473; Symbol type (none) -> Specified Device
Connections:
- net GND: now also R?.1, R?.1
- net DRV2_EN: now reaches U?.6 (EN)
- net PWM2_H: now reaches U?.7 (H_IN)
- net PWM2_L: now reaches U?.8 (L_IN)
- net DRV1_EN: now reaches U?.6 (EN)
- net PWM1_H: now reaches U?.7 (H_IN)
- net PWM1_L: now reaches U?.8 (L_IN)
- new net BS1: R?.2
- new net BS2: R?.2

Commit message: Nightly Update
Parts:
- removed C?: 2.2uF, GENERAL_RCL_SMD:C0805(2012M), symbol 001_Basic_PassiveComponents:101_Capacitor
- removed D?: SS1060HEWS, POWER_DIODE_SMD:SOD-123HE, symbol 002_Basic_SingleSemiconductor:002_Diode_Schottky
- removed R?: 3.3R, GENERAL_RCL_SMD:R0603(1608M), symbol 001_Basic_PassiveComponents:001_Resistor
- added C?: 220nF, 001_GN_RCL_SMD:C0603(1608M), symbol 001_Basic_PassiveComponents:101_Capacitor
- added C? (x2): 2.2uF, 001_GN_RCL_SMD:C0805(2012M), symbol 001_Basic_PassiveComponents:101_Capacitor
- added D?: SS1060HEWS, 002_GN_TWO-PIN_PLASTIC_SMD:SOD-123HE, symbol 002_Basic_SingleSemiconductor:002_Diode_Schottky
- added R?: 3.3R, 001_GN_RCL_SMD:R0603(1608M), symbol 001_Basic_PassiveComponents:001_Resistor
- C?: value 2.2uF -> 220nF; footprint GENERAL_RCL_SMD:C0805(2012M) -> 001_GN_RCL_SMD:C0603(1608M)
- D?: footprint POWER_DIODE_SMD:SOD-123HE -> 002_GN_TWO-PIN_PLASTIC_SMD:SOD-123HE
- R?: footprint GENERAL_RCL_SMD:R0603(1608M) -> 001_GN_RCL_SMD:R0603(1608M)
Connections:
- net GND: now also C?.2, C?.2
- net SW1: now also C?.2
- net Vdrive: now also C?.1, C?.1, D?.2 (Anode)
- net at R?.2: now also C?.1
- net at U?.3 (BST): now also D?.1 (Cathode), R?.1
- net at C?.1: now also R?.2
Other:
- moved on the sheet: C?, D?, R?, U?

Commit message: Complete schematics
Parts:
- gave numbers to parts that had none: 12
Changed lines of the file:
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@@
   (symbol (lib_id "power:Vdrive") (at 86.36 114.3 0) (unit 1)
     (in_bom yes) (on_board yes) (fields_autoplaced)
-    (property "Reference" "#PWR?" (id 0) (at 81.28 118.11 0)
+    (property "Reference" "#PWR0174" (id 0) (at 81.28 118.11 0)
       (effects (font (size 1.27 1.27)) hide)
     )
@@
   (symbol (lib_id "001_Basic_PassiveComponents:101_Capacitor") (at 167.64 55.88 0) (unit 1)
     (in_bom yes) (on_board yes) (fields_autoplaced)
-    (property "Reference" "C?" (id 0) (at 167.64 49.53 0))
+    (property "Reference" "C12" (id 0) (at 167.64 49.53 0))
     (property "Value" "220nF" (id 1) (at 167.64 52.07 0))
     (property "Footprint" "001_GN_RCL_SMD:C0603(1608M)" (id 2) (at 167.64 55.88 0)
@@
   (symbol (lib_id "001_Basic_PassiveComponents:101_Capacitor") (at 86.36 139.7 270) (unit 1)
     (in_bom yes) (on_board yes) (fields_autoplaced)
-    (property "Reference" "C?" (id 0) (at 88.9 138.4299 90)
+    (property "Reference" "C11" (id 0) (at 88.9 138.4299 90)
       (effects (font (size 1.27 1.27)) (justify left))
     )
@@
   (symbol (lib_id "power:GND") (at 86.36 165.1 0) (unit 1)
     (in_bom yes) (on_board yes) (fields_autoplaced)
-    (property "Reference" "#PWR?" (id 0) (at 86.36 171.45 0)
+    (property "Reference" "#PWR0175" (id 0) (at 86.36 171.45 0)
       (effects (font (size 1.27 1.27)) hide)
     )
@@
   (symbol (lib_id "001_Basic_PassiveComponents:001_Resistor") (at 137.16 160.02 0) (unit 1)
     (in_bom yes) (on_board yes) (fields_autoplaced)
-    (property "Reference" "R?" (id 0) (at 137.16 153.67 0))
+    (property "Reference" "R8" (id 0) (at 137.16 153.67 0))
     (property "Value" "0R" (id 1) (at 137.16 156.21 0))
     (property "Footprint" "001_GN_RCL_SMD:R0603(1608M)" (id 2) (at 133.35 156.21 0)
@@
   (symbol (lib_id "001_Basic_PassiveComponents:101_Capacitor") (at 167.64 132.08 0) (unit 1)
     (in_bom yes) (on_board yes) (fields_autoplaced)
-    (property "Reference" "C?" (id 0) (at 167.64 125.73 0))
+    (property "Reference" "C13" (id 0) (at 167.64 125.73 0))
     (property "Value" "220nF" (id 1) (at 167.64 128.27 0))
     (property "Footprint" "001_GN_RCL_SMD:C0603(1608M)" (id 2) (at 167.64 132.08 0)
@@
   (symbol (lib_id "002_Basic_SingleSemiconductor:002_Diode_Schottky") (at 147.32 121.92 90) (unit 1)
     (in_bom yes) (on_board yes) (fields_autoplaced)
-    (property "Reference" "D?" (id 0) (at 149.86 120.6499 90)
+    (property "Reference" "D2" (id 0) (at 149.86 120.6499 90)
       (effects (font (size 1.27 1.27)) (justify right))
     )
@@
   (symbol (lib_id "001_Basic_PassiveComponents:001_Resistor") (at 137.16 83.82 0) (unit 1)
     (in_bom yes) (on_board yes) (fields_autoplaced)
-    (property "Reference" "R?" (id 0) (at 137.16 77.47 0))
+    (property "Reference" "R7" (id 0) (at 137.16 77.47 0))
     (property "Value" "0R" (id 1) (at 137.16 80.01 0))
     (property "Footprint" "001_GN_RCL_SMD:R0603(1608M)" (id 2) (at 133.35 80.01 0)
@@
   (symbol (lib_id "105_IntegratedCircuit_TransistorDriver:DGD05473") (at 137.16 139.7 0) (unit 1)
     (in_bom yes) (on_board yes) (fields_autoplaced)
-    (property "Reference" "U?" (id 0) (at 137.16 125.73 0))
+    (property "Reference" "U3" (id 0) (at 137.16 125.73 0))
     (property "Value" "DGD05473" (id 1) (at 137.16 128.27 0))
     (property "Footprint" "003_GN_SMALL-SEMI_SMD:DFN-10_3030" (id 2) (at 137.16 127 0)
@@
   (symbol (lib_id "power:Vdrive") (at 86.36 38.1 0) (unit 1)
     (in_bom yes) (on_board yes) (fields_autoplaced)
-    (property "Reference" "#PWR?" (id 0) (at 81.28 41.91 0)
+    (property "Reference" "#PWR0172" (id 0) (at 81.28 41.91 0)
       (effects (font (size 1.27 1.27)) hide)
     )
@@
   (symbol (lib_id "001_Basic_PassiveComponents:101_Capacitor") (at 86.36 63.5 270) (unit 1)
     (in_bom yes) (on_board yes) (fields_autoplaced)
-    (property "Reference" "C?" (id 0) (at 88.9 62.2299 90)
+    (property "Reference" "C10" (id 0) (at 88.9 62.2299 90)
       (effects (font (size 1.27 1.27)) (justify left))
     )
@@
   (symbol (lib_id "105_IntegratedCircuit_TransistorDriver:DGD05473") (at 137.16 63.5 0) (unit 1)
     (in_bom yes) (on_board yes) (fields_autoplaced)
-    (property "Reference" "U?" (id 0) (at 137.16 49.53 0))
+    (property "Reference" "U2" (id 0) (at 137.16 49.53 0))
     (property "Value" "DGD05473" (id 1) (at 137.16 52.07 0))
     (property "Footprint" "003_GN_SMALL-SEMI_SMD:DFN-10_3030" (id 2) (at 137.16 50.8 0)
@@
   (symbol (lib_id "001_Basic_PassiveComponents:001_Resistor") (at 154.94 55.88 0) (unit 1)
     (in_bom yes) (on_board yes) (fields_autoplaced)
-    (property "Reference" "R?" (id 0) (at 154.94 49.53 0))
+    (property "Reference" "R9" (id 0) (at 154.94 49.53 0))
     (property "Value" "3.3R" (id 1) (at 154.94 52.07 0))
     (property "Footprint" "001_GN_RCL_SMD:R0603(1608M)" (id 2) (at 151.13 52.07 0)
@@
   (symbol (lib_id "001_Basic_PassiveComponents:001_Resistor") (at 154.94 132.08 0) (unit 1)
     (in_bom yes) (on_board yes) (fields_autoplaced)
-    (property "Reference" "R?" (id 0) (at 154.94 125.73 0))
+    (property "Reference" "R10" (id 0) (at 154.94 125.73 0))
     (property "Value" "3.3R" (id 1) (at 154.94 128.27 0))
     (property "Footprint" "001_GN_RCL_SMD:R0603(1608M)" (id 2) (at 151.13 128.27 0)
@@
   (symbol (lib_id "002_Basic_SingleSemiconductor:002_Diode_Schottky") (at 147.32 45.72 90) (unit 1)
     (in_bom yes) (on_board yes) (fields_autoplaced)
-    (property "Reference" "D?" (id 0) (at 149.86 44.4499 90)
+    (property "Reference" "D1" (id 0) (at 149.86 44.4499 90)
       (effects (font (size 1.27 1.27)) (justify right))
     )
@@
   (symbol (lib_id "power:GND") (at 86.36 88.9 0) (unit 1)
     (in_bom yes) (on_board yes) (fields_autoplaced)
-    (property "Reference" "#PWR?" (id 0) (at 86.36 95.25 0)
-      (effects (font (size 1.27 1.27)) hide)
-    )
+    (property "Reference" "#PWR0173" (id 0) (at 86.36 95.25 0)
+      (effects (font (size 1.27 1.27)) hide)
+    )
