File: hardware/Main_Switch.kicad_sch (KiCad schematic)
At the start: 16 parts

Commit message: Nightly update
Parts:
- removed R? (x4): 10kR, GENERAL_RCL_SMD:R0603(1608M), symbol Basic_passive_components:Resistor
- removed R? (x2): 0R, GENERAL_RCL_SMD:R0402(1005M), symbol Basic_passive_components:Resistor
- removed R? (x3): 5.1R, GENERAL_RCL_SMD:R0603(1608M), symbol Basic_passive_components:Resistor
- added C? (x2): 1nF, 001_GN_RCL_SMD:C0603(1608M), symbol 001_Basic_PassiveComponents:101_Capacitor
- added C? (x2): 100uF, 007_GN_POLAR-CAP_SMD:CL-0810, symbol 001_Basic_PassiveComponents:102_PolarCapacitor
- added R? (x4): 0R, 001_GN_RCL_SMD:R0402(1005M), symbol 001_Basic_PassiveComponents:001_Resistor
- added R? (x4): 10kR, 001_GN_RCL_SMD:R0402(1005M), symbol 001_Basic_PassiveComponents:001_Resistor
- added R? (x2): 22R, 001_GN_RCL_SMD:R0603(1608M), symbol 001_Basic_PassiveComponents:001_Resistor
- added R? (x3): 5.1R, 001_GN_RCL_SMD:R0603(1608M), symbol 001_Basic_PassiveComponents:001_Resistor
- added R?: 10mR, 001_GN_RCL_SMD:R2512(6332M), symbol 001_Basic_PassiveComponents:001_Resistor
- L?: value 202_PowerChoke -> 4.7uH; footprint POWER_INDUCTOR_SMD:MC-1770 -> 008_GN_POWER-CHOKE_SMD:MC-1265
- R?: footprint GENERAL_RCL_SMD:R2512(6332M) -> 001_GN_RCL_SMD:R2512(6332M); symbol Basic_passive_components:Resistor -> 001_Basic_PassiveComponents:001_Resistor; Symbol type (none) -> Alternate Source
- R?: footprint GENERAL_RCL_SMD:R0603(1608M) -> 001_GN_RCL_SMD:R0603(1608M); symbol Basic_passive_components:Resistor -> 001_Basic_PassiveComponents:001_Resistor; Symbol type (none) -> Alternate Source
Connections:
- net BG1: now also R?.1
- net BG2: now also R?.2
- net GND: now also R?.1, C?.2, C?.2, R?.1, R?.1, R?.1, R?.2, R?.2; no longer Q?.S (Source), Q?.S (Source)
- net SW1: now also C?.2, R?.1
- net SW2: now also L?.2, C?.2, R?.1; no longer R?.2
- net TG1: now also R?.1
- net VDC: now also C?.1, C?.1
- net at Q?.G (Gate): now also R?.1, R?.2
- net at Q?.G (Gate): now also R?.2, R?.2 (x2)
- net at Q?.G (Gate), R?.1: now also R?.2
- new net: C?.1, R?.2 (x2)
- new net BS1: Q?.S (Source), R?.1, R?.2, R?.2
- new net BS2: Q?.S (Source), R?.1, R?.2, R?.2
- new net CS1_N: R?.1
- new net CS1_P: R?.1
- new net CS2_N: R?.1
- new net CS2_P: R?.1
Other:
- moved on the sheet: L?, R?

Commit message: Update schematics
Parts:
- C? (x2): footprint 001_GN_RCL_SMD:C0603(1608M) -> 001_GN_RCL_SMD:C0805(2012M)
- R? (x2): footprint 001_GN_RCL_SMD:R0603(1608M) -> 001_GN_RCL_SMD:R0805(2012M)
Changed lines of the file:
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@@
       (effects (font (size 1.27 1.27)) (justify right))
     )
-    (property "Footprint" "001_GN_RCL_SMD:C0603(1608M)" (id 2) (at 127 106.68 0)
+    (property "Footprint" "001_GN_RCL_SMD:C0805(2012M)" (id 2) (at 127 106.68 0)
       (effects (font (size 1.27 1.27)) hide)
     )
@@
       (effects (font (size 1.27 1.27)) (justify right))
     )
-    (property "Footprint" "001_GN_RCL_SMD:R0603(1608M)" (id 2) (at 123.19 130.81 0)
+    (property "Footprint" "001_GN_RCL_SMD:R0805(2012M)" (id 2) (at 123.19 130.81 0)
       (effects (font (size 1.27 1.27)) hide)
     )
@@
       (effects (font (size 1.27 1.27)) (justify right))
     )
-    (property "Footprint" "001_GN_RCL_SMD:C0603(1608M)" (id 2) (at 152.4 106.68 0)
+    (property "Footprint" "001_GN_RCL_SMD:C0805(2012M)" (id 2) (at 152.4 106.68 0)
       (effects (font (size 1.27 1.27)) hide)
     )
@@
       (effects (font (size 1.27 1.27)) (justify right))
     )
-    (property "Footprint" "001_GN_RCL_SMD:R0603(1608M)" (id 2) (at 148.59 130.81 0)
-      (effects (font (size 1.27 1.27)) hide)
-    )
+    (property "Footprint" "001_GN_RCL_SMD:R0805(2012M)" (id 2) (at 148.59 130.81 0)
+      (effects (font (size 1.27 1.27)) hide)
+    )

Commit message: Complete schematics
Parts:
- gave numbers to parts that had none: 25
Changed lines of the file:
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@@
   (symbol (lib_id "001_Basic_PassiveComponents:101_Capacitor") (at 127 106.68 90) (unit 1)
     (in_bom yes) (on_board yes) (fields_autoplaced)
-    (property "Reference" "C?" (id 0) (at 129.54 105.4099 90)
+    (property "Reference" "C15" (id 0) (at 129.54 105.4099 90)
       (effects (font (size 1.27 1.27)) (justify right))
     )
@@
   (symbol (lib_id "202_Power_Transistor:NTMFS5C670NL") (at 177.8 101.6 0) (mirror y) (unit 1)
     (in_bom yes) (on_board yes) (fields_autoplaced)
-    (property "Reference" "Q?" (id 0) (at 174.625 102.87 0))
+    (property "Reference" "Q4" (id 0) (at 174.625 102.87 0))
     (property "Value" "NTMFS5C670NL" (id 1) (at 167.894 100.33 0))
     (property "Footprint" "103_SP_POWER_TRANSISTOR_SMD:SON-6050-FET" (id 2) (at 151.13 97.79 0)
@@
   (symbol (lib_id "001_Basic_PassiveComponents:102_PolarCapacitor") (at 127 63.5 270) (unit 1)
     (in_bom yes) (on_board yes) (fields_autoplaced)
-    (property "Reference" "C?" (id 0) (at 129.54 62.2299 90)
+    (property "Reference" "C14" (id 0) (at 129.54 62.2299 90)
       (effects (font (size 1.27 1.27)) (justify left))
     )
@@
   (symbol (lib_id "001_Basic_PassiveComponents:001_Resistor") (at 86.36 129.54 0) (unit 1)
     (in_bom yes) (on_board yes) (fields_autoplaced)
-    (property "Reference" "R?" (id 0) (at 86.36 123.19 0))
+    (property "Reference" "R13" (id 0) (at 86.36 123.19 0))
     (property "Value" "0R" (id 1) (at 86.36 125.73 0))
     (property "Footprint" "001_GN_RCL_SMD:R0402(1005M)" (id 2) (at 82.55 125.73 0)
@@
   (symbol (lib_id "001_Basic_PassiveComponents:001_Resistor") (at 86.36 144.78 0) (unit 1)
     (in_bom yes) (on_board yes) (fields_autoplaced)
-    (property "Reference" "R?" (id 0) (at 86.36 138.43 0))
+    (property "Reference" "R14" (id 0) (at 86.36 138.43 0))
     (property "Value" "0R" (id 1) (at 86.36 140.97 0))
     (property "Footprint" "001_GN_RCL_SMD:R0402(1005M)" (id 2) (at 82.55 140.97 0)
@@
   (symbol (lib_id "001_Basic_PassiveComponents:001_Resistor") (at 93.98 71.12 90) (unit 1)
     (in_bom yes) (on_board yes) (fields_autoplaced)
-    (property "Reference" "R?" (id 0) (at 96.52 69.8499 90)
+    (property "Reference" "R15" (id 0) (at 96.52 69.8499 90)
       (effects (font (size 1.27 1.27)) (justify right))
     )
@@
   (symbol (lib_id "001_Basic_PassiveComponents:001_Resistor") (at 127 127 90) (unit 1)
     (in_bom yes) (on_board yes) (fields_autoplaced)
-    (property "Reference" "R?" (id 0) (at 129.54 125.7299 90)
+    (property "Reference" "R18" (id 0) (at 129.54 125.7299 90)
       (effects (font (size 1.27 1.27)) (justify right))
     )
@@
   (symbol (lib_id "001_Basic_PassiveComponents:101_Capacitor") (at 152.4 106.68 90) (unit 1)
     (in_bom yes) (on_board yes) (fields_autoplaced)
-    (property "Reference" "C?" (id 0) (at 154.94 105.4099 90)
+    (property "Reference" "C17" (id 0) (at 154.94 105.4099 90)
       (effects (font (size 1.27 1.27)) (justify right))
     )
@@
   (symbol (lib_id "001_Basic_PassiveComponents:001_Resistor") (at 83.82 101.6 0) (unit 1)
     (in_bom yes) (on_board yes) (fields_autoplaced)
-    (property "Reference" "R?" (id 0) (at 83.82 95.25 0))
+    (property "Reference" "R12" (id 0) (at 83.82 95.25 0))
     (property "Value" "5.1R" (id 1) (at 83.82 97.79 0))
     (property "Footprint" "001_GN_RCL_SMD:R0603(1608M)" (id 2) (at 80.01 97.79 0)
@@
   (symbol (lib_id "001_Basic_PassiveComponents:001_Resistor") (at 195.58 101.6 0) (unit 1)
     (in_bom yes) (on_board yes) (fields_autoplaced)
-    (property "Reference" "R?" (id 0) (at 195.58 95.25 0))
+    (property "Reference" "R26" (id 0) (at 195.58 95.25 0))
     (property "Value" "5.1R" (id 1) (at 195.58 97.79 0))
     (property "Footprint" "001_GN_RCL_SMD:R0603(1608M)" (id 2) (at 191.77 97.79 0)
@@
   (symbol (lib_id "001_Basic_PassiveComponents:001_Resistor") (at 152.4 127 90) (unit 1)
     (in_bom yes) (on_board yes) (fields_autoplaced)
-    (property "Reference" "R?" (id 0) (at 154.94 125.7299 90)
+    (property "Reference" "R19" (id 0) (at 154.94 125.7299 90)
       (effects (font (size 1.27 1.27)) (justify right))
     )
@@
   (symbol (lib_id "202_Power_Transistor:NTMFS5C670NL") (at 101.6 63.5 0) (unit 1)
     (in_bom yes) (on_board yes) (fields_autoplaced)
-    (property "Reference" "Q?" (id 0) (at 104.775 64.77 0))
+    (property "Reference" "Q1" (id 0) (at 104.775 64.77 0))
     (property "Value" "NTMFS5C670NL" (id 1) (at 111.506 62.23 0))
     (property "Footprint" "103_SP_POWER_TRANSISTOR_SMD:SON-6050-FET" (id 2) (at 128.27 59.69 0)
@@
   (symbol (lib_id "202_Power_Transistor:NTMFS5C670NL") (at 177.8 63.5 0) (mirror y) (unit 1)
     (in_bom yes) (on_board yes) (fields_autoplaced)
-    (property "Reference" "Q?" (id 0) (at 174.625 64.77 0))
+    (property "Reference" "Q3" (id 0) (at 174.625 64.77 0))
     (property "Value" "NTMFS5C670NL" (id 1) (at 167.894 62.23 0))
     (property "Footprint" "103_SP_POWER_TRANSISTOR_SMD:SON-6050-FET" (id 2) (at 151.13 59.69 0)
@@
   (symbol (lib_id "001_Basic_PassiveComponents:001_Resistor") (at 193.04 132.08 0) (mirror y) (unit 1)
     (in_bom yes) (on_board yes) (fields_autoplaced)
-    (property "Reference" "R?" (id 0) (at 193.04 125.73 0))
+    (property "Reference" "R23" (id 0) (at 193.04 125.73 0))
     (property "Value" "0R" (id 1) (at 193.04 128.27 0))
     (property "Footprint" "001_GN_RCL_SMD:R0402(1005M)" (id 2) (at 196.85 128.27 0)
@@
   (symbol (lib_id "001_Basic_PassiveComponents:102_PolarCapacitor") (at 152.4 63.5 270) (unit 1)
     (in_bom yes) (on_board yes) (fields_autoplaced)
-    (property "Reference" "C?" (id 0) (at 154.94 62.2299 90)
+    (property "Reference" "C16" (id 0) (at 154.94 62.2299 90)
       (effects (font (size 1.27 1.27)) (justify left))
     )
@@
   (symbol (lib_id "202_Power_Transistor:NTMFS5C670NL") (at 101.6 101.6 0) (unit 1)
     (in_bom yes) (on_board yes) (fields_autoplaced)
-    (property "Reference" "Q?" (id 0) (at 104.775 102.87 0))
+    (property "Reference" "Q2" (id 0) (at 104.775 102.87 0))
     (property "Value" "NTMFS5C670NL" (id 1) (at 111.506 100.33 0))
     (property "Footprint" "103_SP_POWER_TRANSISTOR_SMD:SON-6050-FET" (id 2) (at 128.27 97.79 0)
@@
   (symbol (lib_id "001_Basic_PassiveComponents:202_PowerChoke") (at 139.7 88.9 0) (unit 1)
     (in_bom yes) (on_board yes) (fields_autoplaced)
-    (property "Reference" "L?" (id 0) (at 135.255 91.44 0))
+    (property "Reference" "L1" (id 0) (at 135.255 91.44 0))
     (property "Value" "4.7uH" (id 1) (at 139.7 86.36 0))
     (property "Footprint" "008_GN_POWER-CHOKE_SMD:MC-1265" (id 2) (at 139.7 88.9 0)
@@
   (symbol (lib_id "001_Basic_PassiveComponents:001_Resistor") (at 187.96 109.22 90) (unit 1)
     (in_bom yes) (on_board yes) (fields_autoplaced)
-    (property "Reference" "R?" (id 0) (at 190.5 107.9499 90)
+    (property "Reference" "R22" (id 0) (at 190.5 107.9499 90)
       (effects (font (size 1.27 1.27)) (justify right))
     )
@@
   (symbol (lib_id "001_Basic_PassiveComponents:001_Resistor") (at 193.04 147.32 0) (mirror y) (unit 1)
     (in_bom yes) (on_board yes) (fields_autoplaced)
-    (property "Reference" "R?" (id 0) (at 193.04 140.97 0))
+    (property "Reference" "R24" (id 0) (at 193.04 140.97 0))
     (property "Value" "0R" (id 1) (at 193.04 143.51 0))
     (property "Footprint" "001_GN_RCL_SMD:R0402(1005M)" (id 2) (at 196.85 143.51 0)
@@
   (symbol (lib_id "001_Basic_PassiveComponents:001_Resistor") (at 177.8 139.7 90) (unit 1)
     (in_bom yes) (on_board yes) (fields_autoplaced)
-    (property "Reference" "R?" (id 0) (at 180.34 138.4299 90)
+    (property "Reference" "R20" (id 0) (at 180.34 138.4299 90)
       (effects (font (size 1.27 1.27)) (justify right))
     )
@@
   (symbol (lib_id "001_Basic_PassiveComponents:001_Resistor") (at 187.96 71.12 90) (unit 1)
     (in_bom yes) (on_board yes) (fields_autoplaced)
-    (property "Reference" "R?" (id 0) (at 190.5 69.8499 90)
+    (property "Reference" "R21" (id 0) (at 190.5 69.8499 90)
       (effects (font (size 1.27 1.27)) (justify right))
     )
@@
   (symbol (lib_id "001_Basic_PassiveComponents:001_Resistor") (at 195.58 63.5 0) (unit 1)
     (in_bom yes) (on_board yes) (fields_autoplaced)
-    (property "Reference" "R?" (id 0) (at 195.58 57.15 0))
+    (property "Reference" "R25" (id 0) (at 195.58 57.15 0))
     (property "Value" "5.1R" (id 1) (at 195.58 59.69 0))
     (property "Footprint" "001_GN_RCL_SMD:R0603(1608M)" (id 2) (at 191.77 59.69 0)
@@
   (symbol (lib_id "001_Basic_PassiveComponents:001_Resistor") (at 101.6 137.16 90) (unit 1)
     (in_bom yes) (on_board yes) (fields_autoplaced)
-    (property "Reference" "R?" (id 0) (at 104.14 135.8899 90)
+    (property "Reference" "R17" (id 0) (at 104.14 135.8899 90)
       (effects (font (size 1.27 1.27)) (justify right))
     )
@@
   (symbol (lib_id "001_Basic_PassiveComponents:001_Resistor") (at 93.98 109.22 90) (unit 1)
     (in_bom yes) (on_board yes) (fields_autoplaced)
-    (property "Reference" "R?" (id 0) (at 96.52 107.9499 90)
+    (property "Reference" "R16" (id 0) (at 96.52 107.9499 90)
       (effects (font (size 1.27 1.27)) (justify right))
     )
@@
   (symbol (lib_id "001_Basic_PassiveComponents:001_Resistor") (at 83.82 63.5 0) (unit 1)
     (in_bom yes) (on_board yes) (fields_autoplaced)
-    (property "Reference" "R?" (id 0) (at 83.82 57.15 0))
+    (property "Reference" "R11" (id 0) (at 83.82 57.15 0))
     (property "Value" "5.1R" (id 1) (at 83.82 59.69 0))
     (property "Footprint" "001_GN_RCL_SMD:R0603(1608M)" (id 2) (at 80.01 59.69 0)
